File: pcb/fuse.sch (KiCad schematic (older format))
At the start: 65 parts, among them SW0 SW_PUSH, SW1 SW_PUSH, SW10 SW_PUSH, SW11 SW_PUSH, SW12 SW_PUSH, SW13 SW_PUSH, SW14 SW_PUSH, SW15 SW_PUSH, SW2 SW_PUSH, SW20 SW_PUSH, SW21 SW_PUSH, SW22 SW_PUSH, SW23 SW_PUSH, SW24 SW_PUSH, SW25 SW_PUSH, SW3 SW_PUSH, SW30 SW_PUSH, SW31 SW_PUSH, SW32 SW_PUSH, SW33 SW_PUSH, SW34 SW_PUSH, SW35 SW_PUSH, SW4 SW_PUSH, SW40 SW_PUSH, SW41 SW_PUSH, SW42 SW_PUSH, SW43 SW_PUSH, SW44 SW_PUSH, SW45 SW_PUSH, SW5 SW_PUSH, U1 ProMicro, U2 BatteryHole, U3 BatteryHole

Commit message: Remove hotswap to cut down PCB size.
Parts:
- SW0, SW10, SW20, SW30, SW45: footprint fuse-kbd:Choc_Hotswap_Reverse_15 -> fuse-kbd:Choc_Reverse_15
- SW1, SW11, SW12, SW13, SW14, SW15, SW2, SW21, SW22, SW23, SW24, SW25, SW3, SW31, SW32, SW33, SW34, SW35, SW4, SW40, SW41, SW42, SW43, SW44, SW5: footprint fuse-kbd:Choc_Hotswap_Reverse_1 -> fuse-kbd:Choc_Reverse
Changed lines of the file:
@@
 F 0 "SW1" H 2800 1755 50  0000 C CNN
 F 1 "SW_PUSH" H 2800 1664 50  0000 C CNN
-F 2 "fuse-kbd:Choc_Hotswap_Reverse_1" H 2800 1500 50  0001 C CNN
+F 2 "fuse-kbd:Choc_Reverse" H 2800 1500 50  0001 C CNN
 F 3 "" H 2800 1500 50  0000 C CNN
 	1    2800 1500
@@
 F 0 "SW2" H 3800 1755 50  0000 C CNN
 F 1 "SW_PUSH" H 3800 1664 50  0000 C CNN
-F 2 "fuse-kbd:Choc_Hotswap_Reverse_1" H 3800 1500 50  0001 C CNN
+F 2 "fuse-kbd:Choc_Reverse" H 3800 1500 50  0001 C CNN
 F 3 "" H 3800 1500 50  0000 C CNN
 	1    3800 1500
@@
 F 0 "SW3" H 4800 1755 50  0000 C CNN
 F 1 "SW_PUSH" H 4800 1664 50  0000 C CNN
-F 2 "fuse-kbd:Choc_Hotswap_Reverse_1" H 4800 1500 50  0001 C CNN
+F 2 "fuse-kbd:Choc_Reverse" H 4800 1500 50  0001 C CNN
 F 3 "" H 4800 1500 50  0000 C CNN
 	1    4800 1500
@@
 F 0 "SW4" H 5800 1755 50  0000 C CNN
 F 1 "SW_PUSH" H 5800 1664 50  0000 C CNN
-F 2 "fuse-kbd:Choc_Hotswap_Reverse_1" H 5800 1500 50  0001 C CNN
+F 2 "fuse-kbd:Choc_Reverse" H 5800 1500 50  0001 C CNN
 F 3 "" H 5800 1500 50  0000 C CNN
 	1    5800 1500
@@
 F 0 "SW5" H 6800 1755 50  0000 C CNN
 F 1 "SW_PUSH" H 6800 1664 50  0000 C CNN
-F 2 "fuse-kbd:Choc_Hotswap_Reverse_1" H 6800 1500 50  0001 C CNN
+F 2 "fuse-kbd:Choc_Reverse" H 6800 1500 50  0001 C CNN
 F 3 "" H 6800 1500 50  0000 C CNN
 	1    6800 1500
@@
 F 0 "SW0" H 1800 1845 50  0000 C CNN
 F 1 "SW_PUSH" H 1800 1754 50  0000 C CNN
-F 2 "fuse-kbd:Choc_Hotswap_Reverse_15" H 1800 1663 50  0000 C CNN
+F 2 "fuse-kbd:Choc_Reverse_15" H 1800 1663 50  0000 C CNN
 F 3 "" H 1800 1500 50  0000 C CNN
 	1    1800 1500
@@
 F 0 "SW11" H 2800 2755 50  0000 C CNN
 F 1 "SW_PUSH" H 2800 2664 50  0000 C CNN
-F 2 "fuse-kbd:Choc_Hotswap_Reverse_1" H 2800 2500 50  0001 C CNN
+F 2 "fuse-kbd:Choc_Reverse" H 2800 2500 50  0001 C CNN
 F 3 "" H 2800 2500 50  0000 C CNN
 	1    2800 2500
@@
 F 0 "SW12" H 3800 2755 50  0000 C CNN
 F 1 "SW_PUSH" H 3800 2664 50  0000 C CNN
-F 2 "fuse-kbd:Choc_Hotswap_Reverse_1" H 3800 2500 50  0001 C CNN
+F 2 "fuse-kbd:Choc_Reverse" H 3800 2500 50  0001 C CNN
 F 3 "" H 3800 2500 50  0000 C CNN
 	1    3800 2500
@@
 F 0 "SW13" H 4800 2755 50  0000 C CNN
 F 1 "SW_PUSH" H 4800 2664 50  0000 C CNN
-F 2 "fuse-kbd:Choc_Hotswap_Reverse_1" H 4800 2500 50  0001 C CNN
+F 2 "fuse-kbd:Choc_Reverse" H 4800 2500 50  0001 C CNN
 F 3 "" H 4800 2500 50  0000 C CNN
 	1    4800 2500
@@
 F 0 "SW14" H 5800 2755 50  0000 C CNN
 F 1 "SW_PUSH" H 5800 2664 50  0000 C CNN
-F 2 "fuse-kbd:Choc_Hotswap_Reverse_1" H 5800 2500 50  0001 C CNN
+F 2 "fuse-kbd:Choc_Reverse" H 5800 2500 50  0001 C CNN
 F 3 "" H 5800 2500 50  0000 C CNN
 	1    5800 2500
@@
 F 0 "SW15" H 6800 2755 50  0000 C CNN
 F 1 "SW_PUSH" H 6800 2664 50  0000 C CNN
-F 2 "fuse-kbd:Choc_Hotswap_Reverse_1" H 6800 2500 50  0001 C CNN
+F 2 "fuse-kbd:Choc_Reverse" H 6800 2500 50  0001 C CNN
 F 3 "" H 6800 2500 50  0000 C CNN
 	1    6800 2500
@@
 F 0 "SW10" H 1800 2755 50  0000 C CNN
 F 1 "SW_PUSH" H 1800 2664 50  0000 C CNN
-F 2 "fuse-kbd:Choc_Hotswap_Reverse_15" H 1800 2500 50  0001 C CNN
+F 2 "fuse-kbd:Choc_Reverse_15" H 1800 2500 50  0001 C CNN
 F 3 "" H 1800 2500 50  0000 C CNN
 	1    1800 2500
@@
 F 0 "SW21" H 2800 3755 50  0000 C CNN
 F 1 "SW_PUSH" H 2800 3664 50  0000 C CNN
-F 2 "fuse-kbd:Choc_Hotswap_Reverse_1" H 2800 3500 50  0001 C CNN
+F 2 "fuse-kbd:Choc_Reverse" H 2800 3500 50  0001 C CNN
 F 3 "" H 2800 3500 50  0000 C CNN
 	1    2800 3500
@@
 F 0 "SW22" H 3800 3755 50  0000 C CNN
 F 1 "SW_PUSH" H 3800 3664 50  0000 C CNN
-F 2 "fuse-kbd:Choc_Hotswap_Reverse_1" H 3800 3500 50  0001 C CNN
+F 2 "fuse-kbd:Choc_Reverse" H 3800 3500 50  0001 C CNN
 F 3 "" H 3800 3500 50  0000 C CNN
 	1    3800 3500
@@
 F 0 "SW23" H 4800 3755 50  0000 C CNN
 F 1 "SW_PUSH" H 4800 3664 50  0000 C CNN
-F 2 "fuse-kbd:Choc_Hotswap_Reverse_1" H 4800 3500 50  0001 C CNN
+F 2 "fuse-kbd:Choc_Reverse" H 4800 3500 50  0001 C CNN
 F 3 "" H 4800 3500 50  0000 C CNN
 	1    4800 3500
@@
 F 0 "SW24" H 5800 3755 50  0000 C CNN
 F 1 "SW_PUSH" H 5800 3664 50  0000 C CNN
-F 2 "fuse-kbd:Choc_Hotswap_Reverse_1" H 5800 3500 50  0001 C CNN
+F 2 "fuse-kbd:Choc_Reverse" H 5800 3500 50  0001 C CNN
 F 3 "" H 5800 3500 50  0000 C CNN
 	1    5800 3500
@@
 F 0 "SW25" H 6800 3755 50  0000 C CNN
 F 1 "SW_PUSH" H 6800 3664 50  0000 C CNN
-F 2 "fuse-kbd:Choc_Hotswap_Reverse_1" H 6800 3500 50  0001 C CNN
+F 2 "fuse-kbd:Choc_Reverse" H 6800 3500 50  0001 C CNN
 F 3 "" H 6800 3500 50  0000 C CNN
 	1    6800 3500
@@
 F 0 "SW20" H 1800 3755 50  0000 C CNN
 F 1 "SW_PUSH" H 1800 3664 50  0000 C CNN
-F 2 "fuse-kbd:Choc_Hotswap_Reverse_15" H 1800 3500 50  0001 C CNN
+F 2 "fuse-kbd:Choc_Reverse_15" H 1800 3500 50  0001 C CNN
 F 3 "" H 1800 3500 50  0000 C CNN
 	1    1800 3500
@@
 F 0 "SW31" H 2800 4755 50  0000 C CNN
 F 1 "SW_PUSH" H 2800 4664 50  0000 C CNN
-F 2 "fuse-kbd:Choc_Hotswap_Reverse_1" H 2800 4500 50  0001 C CNN
+F 2 "fuse-kbd:Choc_Reverse" H 2800 4500 50  0001 C CNN
 F 3 "" H 2800 4500 50  0000 C CNN
 	1    2800 4500
@@
 F 0 "SW32" H 3800 4755 50  0000 C CNN
 F 1 "SW_PUSH" H 3800 4664 50  0000 C CNN
-F 2 "fuse-kbd:Choc_Hotswap_Reverse_1" H 3800 4500 50  0001 C CNN
+F 2 "fuse-kbd:Choc_Reverse" H 3800 4500 50  0001 C CNN
 F 3 "" H 3800 4500 50  0000 C CNN
 	1    3800 4500
@@
 F 0 "SW33" H 4800 4755 50  0000 C CNN
 F 1 "SW_PUSH" H 4800 4664 50  0000 C CNN
-F 2 "fuse-kbd:Choc_Hotswap_Reverse_1" H 4800 4500 50  0001 C CNN
+F 2 "fuse-kbd:Choc_Reverse" H 4800 4500 50  0001 C CNN
 F 3 "" H 4800 4500 50  0000 C CNN
 	1    4800 4500
@@
 F 0 "SW34" H 5800 4755 50  0000 C CNN
 F 1 "SW_PUSH" H 5800 4664 50  0000 C CNN
-F 2 "fuse-kbd:Choc_Hotswap_Reverse_1" H 5800 4500 50  0001 C CNN
+F 2 "fuse-kbd:Choc_Reverse" H 5800 4500 50  0001 C CNN
 F 3 "" H 5800 4500 50  0000 C CNN
 	1    5800 4500
@@
 F 0 "SW35" H 6800 4755 50  0000 C CNN
 F 1 "SW_PUSH" H 6800 4664 50  0000 C CNN
-F 2 "fuse-kbd:Choc_Hotswap_Reverse_1" H 6800 4500 50  0001 C CNN
+F 2 "fuse-kbd:Choc_Reverse" H 6800 4500 50  0001 C CNN
 F 3 "" H 6800 4500 50  0000 C CNN
 	1    6800 4500
@@
 F 0 "SW30" H 1800 4755 50  0000 C CNN
 F 1 "SW_PUSH" H 1800 4664 50  0000 C CNN
-F 2 "fuse-kbd:Choc_Hotswap_Reverse_15" H 1800 4500 50  0001 C CNN
+F 2 "fuse-kbd:Choc_Reverse_15" H 1800 4500 50  0001 C CNN
 F 3 "" H 1800 4500 50  0000 C CNN
 	1    1800 4500
@@
 F 0 "SW42" H 3800 5755 50  0000 C CNN
 F 1 "SW_PUSH" H 3800 5664 50  0000 C CNN
-F 2 "fuse-kbd:Choc_Hotswap_Reverse_1" H 3800 5500 50  0001 C CNN
+F 2 "fuse-kbd:Choc_Reverse" H 3800 5500 50  0001 C CNN
 F 3 "" H 3800 5500 50  0000 C CNN
 	1    3800 5500
@@
 F 0 "SW43" H 4800 5755 50  0000 C CNN
 F 1 "SW_PUSH" H 4800 5664 50  0000 C CNN
-F 2 "fuse-kbd:Choc_Hotswap_Reverse_1" H 4800 5500 50  0001 C CNN
+F 2 "fuse-kbd:Choc_Reverse" H 4800 5500 50  0001 C CNN
 F 3 "" H 4800 5500 50  0000 C CNN
 	1    4800 5500
@@
 F 0 "SW44" H 5800 5755 50  0000 C CNN
 F 1 "SW_PUSH" H 5800 5664 50  0000 C CNN
-F 2 "fuse-kbd:Choc_Hotswap_Reverse_1" H 5800 5500 50  0001 C CNN
+F 2 "fuse-kbd:Choc_Reverse" H 5800 5500 50  0001 C CNN
 F 3 "" H 5800 5500 50  0000 C CNN
 	1    5800 5500
@@
 F 0 "SW45" H 6800 5755 50  0000 C CNN
 F 1 "SW_PUSH" H 6800 5664 50  0000 C CNN
-F 2 "fuse-kbd:Choc_Hotswap_Reverse_15" H 6800 5500 50  0001 C CNN
+F 2 "fuse-kbd:Choc_Reverse_15" H 6800 5500 50  0001 C CNN
 F 3 "" H 6800 5500 50  0000 C CNN
 	1    6800 5500
@@
 F 0 "SW40" H 1800 5755 50  0000 C CNN
 F 1 "SW_PUSH" H 1800 5664 50  0000 C CNN
-F 2 "fuse-kbd:Choc_Hotswap_Reverse_1" H 1800 5500 50  0001 C CNN
+F 2 "fuse-kbd:Choc_Reverse" H 1800 5500 50  0001 C CNN
 F 3 "" H 1800 5500 50  0000 C CNN
 	1    1800 5500
@@
 F 0 "SW41" H 2800 5755 50  0000 C CNN
 F 1 "SW_PUSH" H 2800 5664 50  0000 C CNN
-F 2 "fuse-kbd:Choc_Hotswap_Reverse_1" H 2800 5500 50  0001 C CNN
+F 2 "fuse-kbd:Choc_Reverse" H 2800 5500 50  0001 C CNN
 F 3 "" H 2800 5500 50  0000 C CNN
 	1    2800 5500

Commit message: fix reset pin and footprints
Parts:
- removed U2: BatteryHole, fuse-kbd:BatteryPins, symbol Fuse-kbd:BatteryHole
- added U4: BatteryHole, fuse-kbd:BatteryPins, symbol Fuse-kbd:BatteryHole
Connections:
- net B+: now also U4.1; no longer Power1.2
- net B-: now also Power1.1
- net RESET: now also U1.22 (RST); no longer U1.24 (RAW)
- net at U3.1: now also Power1.2; no longer Power1.1
Other:
- moved on the sheet: Power1, U3
Changed lines of the file:
@@
 Text GLabel 10100 1250 2    50   Input ~ 0
 B+
-Text GLabel 10100 1350 2    50   Input ~ 0
-RESET
-Text GLabel 10100 1450 2    50   Input ~ 0
-GND
 Text GLabel 9750 4000 2    50   Input ~ 0
 GND
@@
 	1    0    0    -1
 $EndComp
-$Comp
-L Fuse-kbd:PowerSwitch Power1
-U 1 1 6224DB38
-P 9850 3100
-F 0 "Power1" H 9850 3445 50  0000 C CNN
-F 1 "SW_PUSH" H 9850 3354 50  0000 C CNN
-F 2 "fuse-kbd:EG1218" H 9850 3263 50  0001 C CNN
-F 3 "" H 9850 3100 50  0000 C CNN
-	1    9850 3100
-	1    0    0    -1
-$EndComp
-Text GLabel 9000 3100 0    50   Input ~ 0
+Text GLabel 9550 2950 0    50   Input ~ 0
 B-
-Text GLabel 9850 3300 2    50   Input ~ 0
-B+
 Wire Wire Line
 	1500 1500 1500 2500
@@
 Connection ~ 2500 1500
 $Comp
-L Fuse-kbd:BatteryHole U2
-U 1 1 6232876D
-P 9000 3200
-F 0 "U2" H 8871 3076 50  0000 R CNN
-F 1 "BatteryHole" H 8871 3167 50  0000 R CNN
-F 2 "fuse-kbd:BatteryPins" H 9000 3200 50  0001 C CNN
-F 3 "" H 9000 3200 50  0001 C CNN
-	1    9000 3200
-	-1   0    0    1
-$EndComp
-$Comp
 L Fuse-kbd:BatteryHole U3
 U 1 1 62329876
-P 9550 3000
-F 0 "U3" H 9507 3125 50  0000 C CNN
-F 1 "BatteryHole" H 9507 3034 50  0000 C CNN
-F 2 "fuse-kbd:BatteryPins" H 9550 3000 50  0001 C CNN
-F 3 "" H 9550 3000 50  0001 C CNN
-	1    9550 3000
+P 10400 3400
+F 0 "U3" H 10357 3525 50  0000 C CNN
+F 1 "BatteryHole" H 10357 3434 50  0000 C CNN
+F 2 "fuse-kbd:BatteryPins" H 10400 3400 50  0001 C CNN
+F 3 "" H 10400 3400 50  0001 C CNN
+	1    10400 3400
 	1    0    0    -1
 $EndComp
+Text GLabel 10100 1450 2    50   Input ~ 0
+GND
+Text GLabel 10100 1550 2    50   Input ~ 0
+RESET
+$Comp
+L Fuse-kbd:PowerSwitch Power1
+U 1 1 6224DB38
+P 10450 2950
+F 0 "Power1" H 10450 3295 50  0000 C CNN
+F 1 "SW_PUSH" H 10450 3204 50  0000 C CNN
+F 2 "fuse-kbd:EG1218" H 10450 3113 50  0001 C CNN
+F 3 "" H 10450 2950 50  0000 C CNN
+	1    10450 2950
+	1    0    0    -1
+$EndComp
+Wire Wire Line
+	9550 2950 10150 2950
+$Comp
+L Fuse-kbd:BatteryHole U4
+U 1 1 62276F26
+P 10950 3400
+F 0 "U4" H 10907 3525 50  0000 C CNN
+F 1 "BatteryHole" H 10907 3434 50  0000 C CNN
+F 2 "fuse-kbd:BatteryPins" H 10950 3400 50  0001 C CNN
+F 3 "" H 10950 3400 50  0001 C CNN
+	1    10950 3400
+	1    0    0    -1
+$EndComp
+Wire Wire Line
+	10450 3150 10450 3500
+Wire Wire Line
+	10450 3500 10400 3500
+Text GLabel 10950 3700 2    50   Input ~ 0
+B+
+Wire Wire Line
+	10950 3500 10950 3700
 $EndSCHEMATC
